Commit message: Add spawn_entity launch and physics-ready URDF (collision+inertial)
- urdf/zhizhu.urdf: add box collision + inertial so it can be spawned with
  physics for future motion
- worlds/spawn.world: lit world without the model, for spawn_entity
- launch/gazebo_spawn.launch.py: spawn via spawn_entity (see known issue note)

File: src/zhizhu_description/urdf/zhizhu.urdf (robot description, URDF)
Before this commit: robot zhizhu, 1 links, 0 joints
Links:
- link base_link: mass None -> 10.0; geometry collision box size=3.68 1.78 0.894; visual mesh filename=file:///home/khalil/ROS/zhizhu/install/zhizhu_description/s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 scale=0.001 0.001 0.001

Commit message: Stage 1: flip back (feet down) + decompose into body + 6 virtual feet
- body link: single STL as visual, approximate hub box collision
- 6 foot links (red spheres, ESTIMATED positions) fixed to body for ground contact
- flip rpy back to 0 so the suction/foot side faces down

File: src/zhizhu_description/urdf/zhizhu.urdf (robot description, URDF)
Before this commit: robot zhizhu, 1 links, 0 joints
Links:
- removed link base_link
- added link body, mass 10.0; collision box size=0.6 0.8 0.5; visual mesh filename=file:///home/khalil/ROS/zhizhu/install/zhizhu_description/s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 scale=0.001 0.001 0.001
- added link foot_lf, mass 0.5; collision sphere radius=0.08; visual sphere radius=0.08
- added link foot_lm, mass 0.5; collision sphere radius=0.08; visual sphere radius=0.08
- added link foot_lr, mass 0.5; collision sphere radius=0.08; visual sphere radius=0.08
- added link foot_rf, mass 0.5; collision sphere radius=0.08; visual sphere radius=0.08
- added link foot_rm, mass 0.5; collision sphere radius=0.08; visual sphere radius=0.08
- added link foot_rr, mass 0.5; collision sphere radius=0.08; visual sphere radius=0.08
Joints:
- added joint body_to_foot_lf: type fixed, parent body, child foot_lf, origin xyz=-1.2 -0.85 0.05 rpy=0 0 0
- added joint body_to_foot_lm: type fixed, parent body, child foot_lm, origin xyz=0.0 -0.85 0.05 rpy=0 0 0
- added joint body_to_foot_lr: type fixed, parent body, child foot_lr, origin xyz=1.2 -0.85 0.05 rpy=0 0 0
- added joint body_to_foot_rf: type fixed, parent body, child foot_rf, origin xyz=-1.2 0.85 0.05 rpy=0 0 0
- added joint body_to_foot_rm: type fixed, parent body, child foot_rm, origin xyz=0.0 0.85 0.05 rpy=0 0 0
- added joint body_to_foot_rr: type fixed, parent body, child foot_rr, origin xyz=1.2 0.85 0.05 rpy=0 0 0

Commit message: GUI control + box collision + joint damping
- display.launch.py uses joint_state_publisher_gui (sliders to move legs)
- collision geometry changed from mesh to box (less rendering data, addresses
  the RViz tremor)
- joint dynamics damping/friction 0.5 so legs don't swing freely in Gazebo

File: src/zhizhu_description/urdf/zhizhu.urdf (robot description, URDF)
Before this commit: robot zhizhu, 19 links, 18 joints
Links:
- link body: geometry collision box size=0.782 0.700 0.442; visual mesh filename=file:///home/khalil/ROS/zhizhu/install/zhizhu_description/s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
- link lf_coxa: geometry collision box size=0.728 0.377 0.168; visual mesh filename=file:///home/khalil/ROS/zhizhu/install/zhizhu_description/s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
- link lf_femur: geometry collision box size=0.717 0.323 0.495; visual mesh filename=file:///home/khalil/ROS/zhizhu/install/zhizhu_description/s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
- link lf_foot: geometry collision box size=0.203 0.204 0.214; visual mesh filename=file:///home/khalil/ROS/zhizhu/install/zhizhu_description/s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
- link lm_coxa: geometry collision box size=0.723 0.116 0.192; visual mesh filename=file:///home/khalil/ROS/zhizhu/install/zhizhu_description/s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
- link lm_femur: geometry collision box size=0.818 0.111 0.337; visual mesh filename=file:///home/khalil/ROS/zhizhu/install/zhizhu_description/s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
- link lm_foot: geometry collision box size=0.204 0.202 0.209; visual mesh filename=file:///home/khalil/ROS/zhizhu/install/zhizhu_description/s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
- link lr_coxa: geometry collision box size=0.707 0.404 0.165; visual mesh filename=file:///home/khalil/ROS/zhizhu/install/zhizhu_description/s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
- link lr_femur: geometry collision box size=0.755 0.398 0.336; visual mesh filename=file:///home/khalil/ROS/zhizhu/install/zhizhu_description/s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
- link lr_foot: geometry collision box size=0.202 0.204 0.211; visual mesh filename=file:///home/khalil/ROS/zhizhu/install/zhizhu_description/s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
- link rf_coxa: geometry collision box size=0.692 0.404 0.268; visual mesh filename=file:///home/khalil/ROS/zhizhu/install/zhizhu_description/s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
- link rf_femur: geometry collision box size=0.782 0.398 0.204; visual mesh filename=file:///home/khalil/ROS/zhizhu/install/zhizhu_description/s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
- link rf_foot: geometry collision box size=0.203 0.204 0.212; visual mesh filename=file:///home/khalil/ROS/zhizhu/install/zhizhu_description/s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
- link rm_coxa: geometry collision box size=0.728 0.116 0.227; visual mesh filename=file:///home/khalil/ROS/zhizhu/install/zhizhu_description/s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
- link rm_femur: geometry collision box size=0.837 0.111 0.251; visual mesh filename=file:///home/khalil/ROS/zhizhu/install/zhizhu_description/s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
- link rm_foot: geometry collision box size=0.202 0.202 0.215; visual mesh filename=file:///home/khalil/ROS/zhizhu/install/zhizhu_description/s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
- link rr_coxa: geometry collision box size=0.697 0.377 0.338; visual mesh filename=file:///home/khalil/ROS/zhizhu/install/zhizhu_description/s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
- link rr_femur: geometry collision box size=0.792 0.323 0.318; visual mesh filename=file:///home/khalil/ROS/zhizhu/install/zhizhu_description/s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
- link rr_foot: geometry collision box size=0.201 0.204 0.206; visual mesh filename=file:///home/khalil/ROS/zhizhu/install/zhizhu_description/s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

File: src/zhizhu_description/urdf/zhizhu.xacro (robot description, xacro)
@@ -2,34 +2,34 @@
 <robot name="zhizhu" xmlns:xacro="http://www.ros.org/wiki/xacro">
   <material name="zhizhu_gray"><color rgba="0.7 0.7 0.72 1.0"/></material>
-  <xacro:macro name="leg" params="name hip knee ankle">
+  <xacro:macro name="leg" params="name hip knee ankle coxa_box femur_box foot_box">
     <link name="${name}_coxa">
       <visual><geometry><mesh filename="file:///home/khalil/ROS/zhizhu/install/zhizhu_description/share/zhizhu_description/meshes/parts_urdf/${name}_coxa.stl"/></geometry><material name="zhizhu_gray"/></visual>
-      <collision><geometry><mesh filename="file:///home/khalil/ROS/zhizhu/install/zhizhu_description/share/zhizhu_description/meshes/parts_urdf/${name}_coxa.stl"/></geometry></collision>
+      <collision><geometry><box size="${coxa_box}"/></geometry></collision>
       <inertial><mass value="1.5"/><inertia ixx="0.05" ixy="0" ixz="0" iyy="0.05" iyz="0" izz="0.05"/></inertial>
     </link>
     <link name="${name}_femur">
       <visual><geometry><mesh filename="file:///home/khalil/ROS/zhizhu/install/zhizhu_description/share/zhizhu_description/meshes/parts_urdf/${name}_femur.stl"/></geometry><material name="zhizhu_gray"/></visual>
-      <collision><geometry><mesh filename="file:///home/khalil/ROS/zhizhu/install/zhizhu_description/share/zhizhu_description/meshes/parts_urdf/${name}_femur.stl"/></geometry></collision>
+      <collision><geometry><box size="${femur_box}"/></geometry></collision>
       <inertial><mass value="1.2"/><inertia ixx="0.04" ixy="0" ixz="0" iyy="0.04" iyz="0" izz="0.04"/></inertial>
     </link>
     <link name="${name}_foot">
       <visual><geometry><mesh filename="file:///home/khalil/ROS/zhizhu/install/zhizhu_description/share/zhizhu_description/meshes/parts_urdf/${name}_foot.stl"/></geometry><material name="zhizhu_gray"/></visual>
-      <collision><geometry><mesh filename="file:///home/khalil/ROS/zhizhu/install/zhizhu_description/share/zhizhu_description/meshes/parts_urdf/${name}_foot.stl"/></geometry></collision>
+      <collision><geometry><box size="${foot_box}"/></geometry></collision>
       <inertial><mass value="0.8"/><inertia ixx="0.01" ixy="0" ixz="0" iyy="0.01" iyz="0" izz="0.01"/></inertial>
     </link>
-    <joint name="hip_${name}" type="revolute"><parent link="body"/><child link="${name}_coxa"/><origin xyz="${hip}"/><axis xyz="0 0 1"/><limit lower="-1.57" upper="1.57" effort="50" velocity="5"/><dynamics damping="0.1" friction="0.1"/></joint>
-    <joint name="knee_${name}" type="revolute"><parent link="${name}_coxa"/><child link="${name}_femur"/><origin xyz="${knee}"/><axis xyz="0 1 0"/><limit lower="-1.57" upper="1.57" effort="50" velocity="5"/><dynamics damping="0.1" friction="0.1"/></joint>
-    <joint name="ankle_${name}" type="revolute"><parent link="${name}_femur"/><child link="${name}_foot"/><origin xyz="${ankle}"/><axis xyz="0 1 0"/><limit lower="-0.78" upper="0.78" effort="30" velocity="5"/><dynamics damping="0.1" friction="0.1"/></joint>
+    <joint name="hip_${name}" type="revolute"><parent link="body"/><child link="${name}_coxa"/><origin xyz="${hip}"/><axis xyz="0 0 1"/><limit lower="-1.57" upper="1.57" effort="50" velocity="5"/><dynamics damping="0.5" friction="0.5"/></joint>
+    <joint name="knee_${name}" type="revolute"><parent link="${name}_coxa"/><child link="${name}_femur"/><origin xyz="${knee}"/><axis xyz="0 1 0"/><limit lower="-1.57" upper="1.57" effort="50" velocity="5"/><dynamics damping="0.5" friction="0.5"/></joint>
+    <joint name="ankle_${name}" type="revolute"><parent link="${name}_femur"/><child link="${name}_foot"/><origin xyz="${ankle}"/><axis xyz="0 1 0"/><limit lower="-0.78" upper="0.78" effort="30" velocity="5"/><dynamics damping="0.5" friction="0.5"/></joint>
   </xacro:macro>
   <link name="body">
     <visual><geometry><mesh filename="file:///home/khalil/ROS/zhizhu/install/zhizhu_description/share/zhizhu_description/meshes/parts_urdf/body.stl"/></geometry><material name="zhizhu_gray"/></visual>
-    <collision><geometry><mesh filename="file:///home/khalil/ROS/zhizhu/install/zhizhu_description/share/zhizhu_description/meshes/parts_urdf/body.stl"/></geometry></collision>
+    <collision><geometry><box size="0.782 0.700 0.442"/></geometry></collision>
     <inertial><mass value="6.0"/><inertia ixx="0.4" ixy="0" ixz="0" iyy="0.35" iyz="0" izz="0.45"/></inertial>
   </link>
-  <xacro:leg name="rf" hip="0.7292 0.4250 -0.0111" knee="0.6209 0.2902 0.0107" ankle="0.2435 0.1004 -0.0647"/>
-  <xacro:leg name="rm" hip="0.7729 -0.0080 -0.0299" knee="0.6838 -0.0121 -0.1247" ankle="0.2718 -0.0053 -0.0815"/>
-  <xacro:leg name="rr" hip="0.7419 -0.4061 0.0572" knee="0.6345 -0.2340 -0.0648" ankle="0.2428 -0.0751 -0.1039"/>
-  <xacro:leg name="lf" hip="-0.7421 0.4061 -0.0562" knee="-0.5934 0.2340 -0.2338" ankle="-0.2057 0.0751 -0.1656"/>
-  <xacro:leg name="lm" hip="-0.7678 0.0080 -0.0806" knee="-0.6650 0.0121 -0.2024" ankle="-0.2607 0.0053 -0.1121"/>
-  <xacro:leg name="lr" hip="-0.7200 -0.4250 -0.0891" knee="-0.6110 -0.2902 -0.1110" ankle="-0.2262 -0.1004 -0.1111"/>
+  <xacro:leg name="rf" hip="0.7292 0.4250 -0.0111" knee="0.6209 0.2902 0.0107" ankle="0.2435 0.1004 -0.0647" coxa_box="0.692 0.404 0.268" femur_box="0.782 0.398 0.204" foot_box="0.203 0.204 0.212"/>
+  <xacro:leg name="rm" hip="0.7729 -0.0080 -0.0299" knee="0.6838 -0.0121 -0.1247" ankle="0.2718 -0.0053 -0.0815" coxa_box="0.728 0.116 0.227" femur_box="0.837 0.111 0.251" foot_box="0.202 0.202 0.215"/>
+  <xacro:leg name="rr" hip="0.7419 -0.4061 0.0572" knee="0.6345 -0.2340 -0.0648" ankle="0.2428 -0.0751 -0.1039" coxa_box="0.697 0.377 0.338" femur_box="0.792 0.323 0.318" foot_box="0.201 0.204 0.206"/>
+  <xacro:leg name="lf" hip="-0.7421 0.4061 -0.0562" knee="-0.5934 0.2340 -0.2338" ankle="-0.2057 0.0751 -0.1656" coxa_box="0.728 0.377 0.168" femur_box="0.717 0.323 0.495" foot_box="0.203 0.204 0.214"/>
+  <xacro:leg name="lm" hip="-0.7678 0.0080 -0.0806" knee="-0.6650 0.0121 -0.2024" ankle="-0.2607 0.0053 -0.1121" coxa_box="0.723 0.116 0.192" femur_box="0.818 0.111 0.337" foot_box="0.204 0.202 0.209"/>
+  <xacro:leg name="lr" hip="-0.7200 -0.4250 -0.0891" knee="-0.6110 -0.2902 -0.1110" ankle="-0.2262 -0.1004 -0.1111" coxa_box="0.707 0.404 0.165" femur_box="0.755 0.398 0.336" foot_box="0.202 0.204 0.211"/>
 </robot>

Commit message: Use real joint axes computed from leg geometry (hip horizontal, knee/ankle in leg bending plane)
Previous axes (hip=Z, knee=Y) made the joints spin about themselves instead of
bending about the actual hinge. Computed each leg's hip axis (horizontal,
perpendicular to coxa) and knee/ankle axis (normal to the coxa-femur-foot
bending plane) from the STL centroids.

File: src/zhizhu_description/urdf/zhizhu.urdf (robot description, URDF)
Before this commit: robot zhizhu, 19 links, 18 joints
Joints:
- joint ankle_lf: axis 0 1 0 -> -0.3882 -0.9192 0.0654
- joint ankle_lm: axis 0 1 0 -> -0.0130 -0.9998 -0.0173
- joint ankle_lr: axis 0 1 0 -> 0.4406 -0.8932 -0.0896
- joint ankle_rf: axis 0 1 0 -> -0.4145 0.8932 -0.1741
- joint ankle_rm: axis 0 1 0 -> 0.0149 0.9998 -0.0157
- joint ankle_rr: axis 0 1 0 -> 0.3561 0.9192 0.1678
- joint hip_lf: axis 0 0 1 -> 0.3668 0.9303 -0.0000
- joint hip_lm: axis 0 0 1 -> 0.0183 0.9998 -0.0000
- joint hip_lr: axis 0 0 1 -> -0.4290 0.9033 0.0000
- joint hip_rf: axis 0 0 1 -> 0.4234 -0.9059 0.0000
- joint hip_rm: axis 0 0 1 -> -0.0178 -0.9998 0.0000
- joint hip_rr: axis 0 0 1 -> -0.3460 -0.9382 0.0000
- joint knee_lf: axis 0 1 0 -> -0.3882 -0.9192 0.0654
- joint knee_lm: axis 0 1 0 -> -0.0130 -0.9998 -0.0173
- joint knee_lr: axis 0 1 0 -> 0.4406 -0.8932 -0.0896
- joint knee_rf: axis 0 1 0 -> -0.4145 0.8932 -0.1741
- joint knee_rm: axis 0 1 0 -> 0.0149 0.9998 -0.0157
- joint knee_rr: axis 0 1 0 -> 0.3561 0.9192 0.1678

File: src/zhizhu_description/urdf/zhizhu.xacro (robot description, xacro)
@@ -2,5 +2,5 @@
 <robot name="zhizhu" xmlns:xacro="http://www.ros.org/wiki/xacro">
   <material name="zhizhu_gray"><color rgba="0.7 0.7 0.72 1.0"/></material>
-  <xacro:macro name="leg" params="name hip knee ankle coxa_box femur_box foot_box">
+  <xacro:macro name="leg" params="name hip knee ankle hip_axis knee_axis ankle_axis coxa_box femur_box foot_box">
     <link name="${name}_coxa">
       <visual><geometry><mesh filename="file:///home/khalil/ROS/zhizhu/install/zhizhu_description/share/zhizhu_description/meshes/parts_urdf/${name}_coxa.stl"/></geometry><material name="zhizhu_gray"/></visual>
@@ -18,7 +18,7 @@
       <inertial><mass value="0.8"/><inertia ixx="0.01" ixy="0" ixz="0" iyy="0.01" iyz="0" izz="0.01"/></inertial>
     </link>
-    <joint name="hip_${name}" type="revolute"><parent link="body"/><child link="${name}_coxa"/><origin xyz="${hip}"/><axis xyz="0 0 1"/><limit lower="-1.57" upper="1.57" effort="50" velocity="5"/><dynamics damping="0.5" friction="0.5"/></joint>
-    <joint name="knee_${name}" type="revolute"><parent link="${name}_coxa"/><child link="${name}_femur"/><origin xyz="${knee}"/><axis xyz="0 1 0"/><limit lower="-1.57" upper="1.57" effort="50" velocity="5"/><dynamics damping="0.5" friction="0.5"/></joint>
-    <joint name="ankle_${name}" type="revolute"><parent link="${name}_femur"/><child link="${name}_foot"/><origin xyz="${ankle}"/><axis xyz="0 1 0"/><limit lower="-0.78" upper="0.78" effort="30" velocity="5"/><dynamics damping="0.5" friction="0.5"/></joint>
+    <joint name="hip_${name}" type="revolute"><parent link="body"/><child link="${name}_coxa"/><origin xyz="${hip}"/><axis xyz="${hip_axis}"/><limit lower="-1.57" upper="1.57" effort="50" velocity="5"/><dynamics damping="0.5" friction="0.5"/></joint>
+    <joint name="knee_${name}" type="revolute"><parent link="${name}_coxa"/><child link="${name}_femur"/><origin xyz="${knee}"/><axis xyz="${knee_axis}"/><limit lower="-1.57" upper="1.57" effort="50" velocity="5"/><dynamics damping="0.5" friction="0.5"/></joint>
+    <joint name="ankle_${name}" type="revolute"><parent link="${name}_femur"/><child link="${name}_foot"/><origin xyz="${ankle}"/><axis xyz="${ankle_axis}"/><limit lower="-0.78" upper="0.78" effort="30" velocity="5"/><dynamics damping="0.5" friction="0.5"/></joint>
   </xacro:macro>
   <link name="body">
@@ -27,9 +27,9 @@
     <inertial><mass value="6.0"/><inertia ixx="0.4" ixy="0" ixz="0" iyy="0.35" iyz="0" izz="0.45"/></inertial>
   </link>
-  <xacro:leg name="rf" hip="0.7292 0.4250 -0.0111" knee="0.6209 0.2902 0.0107" ankle="0.2435 0.1004 -0.0647" coxa_box="0.692 0.404 0.268" femur_box="0.782 0.398 0.204" foot_box="0.203 0.204 0.212"/>
-  <xacro:leg name="rm" hip="0.7729 -0.0080 -0.0299" knee="0.6838 -0.0121 -0.1247" ankle="0.2718 -0.0053 -0.0815" coxa_box="0.728 0.116 0.227" femur_box="0.837 0.111 0.251" foot_box="0.202 0.202 0.215"/>
-  <xacro:leg name="rr" hip="0.7419 -0.4061 0.0572" knee="0.6345 -0.2340 -0.0648" ankle="0.2428 -0.0751 -0.1039" coxa_box="0.697 0.377 0.338" femur_box="0.792 0.323 0.318" foot_box="0.201 0.204 0.206"/>
-  <xacro:leg name="lf" hip="-0.7421 0.4061 -0.0562" knee="-0.5934 0.2340 -0.2338" ankle="-0.2057 0.0751 -0.1656" coxa_box="0.728 0.377 0.168" femur_box="0.717 0.323 0.495" foot_box="0.203 0.204 0.214"/>
-  <xacro:leg name="lm" hip="-0.7678 0.0080 -0.0806" knee="-0.6650 0.0121 -0.2024" ankle="-0.2607 0.0053 -0.1121" coxa_box="0.723 0.116 0.192" femur_box="0.818 0.111 0.337" foot_box="0.204 0.202 0.209"/>
-  <xacro:leg name="lr" hip="-0.7200 -0.4250 -0.0891" knee="-0.6110 -0.2902 -0.1110" ankle="-0.2262 -0.1004 -0.1111" coxa_box="0.707 0.404 0.165" femur_box="0.755 0.398 0.336" foot_box="0.202 0.204 0.211"/>
+  <xacro:leg name="rf" hip="0.7292 0.4250 -0.0111" knee="0.6209 0.2902 0.0107" ankle="0.2435 0.1004 -0.0647" hip_axis="0.4234 -0.9059 0.0000" knee_axis="-0.4145 0.8932 -0.1741" ankle_axis="-0.4145 0.8932 -0.1741" coxa_box="0.692 0.404 0.268" femur_box="0.782 0.398 0.204" foot_box="0.203 0.204 0.212"/>
+  <xacro:leg name="rm" hip="0.7729 -0.0080 -0.0299" knee="0.6838 -0.0121 -0.1247" ankle="0.2718 -0.0053 -0.0815" hip_axis="-0.0178 -0.9998 0.0000" knee_axis="0.0149 0.9998 -0.0157" ankle_axis="0.0149 0.9998 -0.0157" coxa_box="0.728 0.116 0.227" femur_box="0.837 0.111 0.251" foot_box="0.202 0.202 0.215"/>
+  <xacro:leg name="rr" hip="0.7419 -0.4061 0.0572" knee="0.6345 -0.2340 -0.0648" ankle="0.2428 -0.0751 -0.1039" hip_axis="-0.3460 -0.9382 0.0000" knee_axis="0.3561 0.9192 0.1678" ankle_axis="0.3561 0.9192 0.1678" coxa_box="0.697 0.377 0.338" femur_box="0.792 0.323 0.318" foot_box="0.201 0.204 0.206"/>
+  <xacro:leg name="lf" hip="-0.7421 0.4061 -0.0562" knee="-0.5934 0.2340 -0.2338" ankle="-0.2057 0.0751 -0.1656" hip_axis="0.3668 0.9303 -0.0000" knee_axis="-0.3882 -0.9192 0.0654" ankle_axis="-0.3882 -0.9192 0.0654" coxa_box="0.728 0.377 0.168" femur_box="0.717 0.323 0.495" foot_box="0.203 0.204 0.214"/>
+  <xacro:leg name="lm" hip="-0.7678 0.0080 -0.0806" knee="-0.6650 0.0121 -0.2024" ankle="-0.2607 0.0053 -0.1121" hip_axis="0.0183 0.9998 -0.0000" knee_axis="-0.0130 -0.9998 -0.0173" ankle_axis="-0.0130 -0.9998 -0.0173" coxa_box="0.723 0.116 0.192" femur_box="0.818 0.111 0.337" foot_box="0.204 0.202 0.209"/>
+  <xacro:leg name="lr" hip="-0.7200 -0.4250 -0.0891" knee="-0.6110 -0.2902 -0.1110" ankle="-0.2262 -0.1004 -0.1111" hip_axis="-0.4290 0.9033 0.0000" knee_axis="0.4406 -0.8932 -0.0896" ankle_axis="0.4406 -0.8932 -0.0896" coxa_box="0.707 0.404 0.165" femur_box="0.755 0.398 0.336" foot_box="0.202 0.204 0.211"/>
 </robot>
