Commit message: Flip robot right-side-up (rpy=0) + recompute joint axes (3-point plane normal)
User reported the robot was upside down. Reverted the transform from rpy=pi
(flip Y/Z) to rpy=0 (no flip), which puts the body low and legs up as expected.
Recomputed knee/ankle axes as the normal of the coxa-femur-foot plane.

File: src/zhizhu_description/urdf/zhizhu.urdf (robot description, URDF)
Before this commit: robot zhizhu, 19 links, 18 joints
Joints:
- joint ankle_lf: axis -0.3882 -0.9192 0.0654 -> -0.3882 0.9192 -0.0654; origin xyz=-0.2057 0.0751 -0.1656 -> xyz=-0.2057 -0.0751 0.1656
- joint ankle_lm: axis -0.0130 -0.9998 -0.0173 -> -0.0130 0.9998 0.0173; origin xyz=-0.2607 0.0053 -0.1121 -> xyz=-0.2607 -0.0053 0.1121
- joint ankle_lr: axis 0.4406 -0.8932 -0.0896 -> 0.4406 0.8932 0.0896; origin xyz=-0.2262 -0.1004 -0.1111 -> xyz=-0.2262 0.1004 0.1111
- joint ankle_rf: axis -0.4145 0.8932 -0.1741 -> -0.4145 -0.8932 0.1741; origin xyz=0.2435 0.1004 -0.0647 -> xyz=0.2435 -0.1004 0.0647
- joint ankle_rm: axis 0.0149 0.9998 -0.0157 -> 0.0149 -0.9998 0.0157; origin xyz=0.2718 -0.0053 -0.0815 -> xyz=0.2718 0.0053 0.0815
- joint ankle_rr: axis 0.3561 0.9192 0.1678 -> 0.3561 -0.9192 -0.1678; origin xyz=0.2428 -0.0751 -0.1039 -> xyz=0.2428 0.0751 0.1039
- joint hip_lf: axis 0.3668 0.9303 -0.0000 -> -0.3668 0.9303 0.0000; origin xyz=-0.7421 0.4061 -0.0562 -> xyz=-0.7421 -0.4061 0.0562
- joint hip_lm: axis 0.0183 0.9998 -0.0000 -> -0.0183 0.9998 0.0000; origin xyz=-0.7678 0.0080 -0.0806 -> xyz=-0.7678 -0.0080 0.0806
- joint hip_lr: axis -0.4290 0.9033 0.0000 -> 0.4290 0.9033 -0.0000; origin xyz=-0.7200 -0.4250 -0.0891 -> xyz=-0.7200 0.4250 0.0891
- joint hip_rf: axis 0.4234 -0.9059 0.0000 -> -0.4234 -0.9059 0.0000; origin xyz=0.7292 0.4250 -0.0111 -> xyz=0.7292 -0.4250 0.0111
- joint hip_rm: axis -0.0178 -0.9998 0.0000 -> 0.0178 -0.9998 0.0000; origin xyz=0.7729 -0.0080 -0.0299 -> xyz=0.7729 0.0080 0.0299
- joint hip_rr: axis -0.3460 -0.9382 0.0000 -> 0.3460 -0.9382 0.0000; origin xyz=0.7419 -0.4061 0.0572 -> xyz=0.7419 0.4061 -0.0572
- joint knee_lf: axis -0.3882 -0.9192 0.0654 -> -0.3882 0.9192 -0.0654; origin xyz=-0.5934 0.2340 -0.2338 -> xyz=-0.5934 -0.2340 0.2338
- joint knee_lm: axis -0.0130 -0.9998 -0.0173 -> -0.0130 0.9998 0.0173; origin xyz=-0.6650 0.0121 -0.2024 -> xyz=-0.6650 -0.0121 0.2024
- joint knee_lr: axis 0.4406 -0.8932 -0.0896 -> 0.4406 0.8932 0.0896; origin xyz=-0.6110 -0.2902 -0.1110 -> xyz=-0.6110 0.2902 0.1110
- joint knee_rf: axis -0.4145 0.8932 -0.1741 -> -0.4145 -0.8932 0.1741; origin xyz=0.6209 0.2902 0.0107 -> xyz=0.6209 -0.2902 -0.0107
- joint knee_rm: axis 0.0149 0.9998 -0.0157 -> 0.0149 -0.9998 0.0157; origin xyz=0.6838 -0.0121 -0.1247 -> xyz=0.6838 0.0121 0.1247
- joint knee_rr: axis 0.3561 0.9192 0.1678 -> 0.3561 -0.9192 -0.1678; origin xyz=0.6345 -0.2340 -0.0648 -> xyz=0.6345 0.2340 0.0648

File: src/zhizhu_description/urdf/zhizhu.xacro (robot description, xacro)
@@ -27,9 +27,9 @@
     <inertial><mass value="6.0"/><inertia ixx="0.4" ixy="0" ixz="0" iyy="0.35" iyz="0" izz="0.45"/></inertial>
   </link>
-  <xacro:leg name="rf" hip="0.7292 0.4250 -0.0111" knee="0.6209 0.2902 0.0107" ankle="0.2435 0.1004 -0.0647" hip_axis="0.4234 -0.9059 0.0000" knee_axis="-0.4145 0.8932 -0.1741" ankle_axis="-0.4145 0.8932 -0.1741" coxa_box="0.692 0.404 0.268" femur_box="0.782 0.398 0.204" foot_box="0.203 0.204 0.212"/>
-  <xacro:leg name="rm" hip="0.7729 -0.0080 -0.0299" knee="0.6838 -0.0121 -0.1247" ankle="0.2718 -0.0053 -0.0815" hip_axis="-0.0178 -0.9998 0.0000" knee_axis="0.0149 0.9998 -0.0157" ankle_axis="0.0149 0.9998 -0.0157" coxa_box="0.728 0.116 0.227" femur_box="0.837 0.111 0.251" foot_box="0.202 0.202 0.215"/>
-  <xacro:leg name="rr" hip="0.7419 -0.4061 0.0572" knee="0.6345 -0.2340 -0.0648" ankle="0.2428 -0.0751 -0.1039" hip_axis="-0.3460 -0.9382 0.0000" knee_axis="0.3561 0.9192 0.1678" ankle_axis="0.3561 0.9192 0.1678" coxa_box="0.697 0.377 0.338" femur_box="0.792 0.323 0.318" foot_box="0.201 0.204 0.206"/>
-  <xacro:leg name="lf" hip="-0.7421 0.4061 -0.0562" knee="-0.5934 0.2340 -0.2338" ankle="-0.2057 0.0751 -0.1656" hip_axis="0.3668 0.9303 -0.0000" knee_axis="-0.3882 -0.9192 0.0654" ankle_axis="-0.3882 -0.9192 0.0654" coxa_box="0.728 0.377 0.168" femur_box="0.717 0.323 0.495" foot_box="0.203 0.204 0.214"/>
-  <xacro:leg name="lm" hip="-0.7678 0.0080 -0.0806" knee="-0.6650 0.0121 -0.2024" ankle="-0.2607 0.0053 -0.1121" hip_axis="0.0183 0.9998 -0.0000" knee_axis="-0.0130 -0.9998 -0.0173" ankle_axis="-0.0130 -0.9998 -0.0173" coxa_box="0.723 0.116 0.192" femur_box="0.818 0.111 0.337" foot_box="0.204 0.202 0.209"/>
-  <xacro:leg name="lr" hip="-0.7200 -0.4250 -0.0891" knee="-0.6110 -0.2902 -0.1110" ankle="-0.2262 -0.1004 -0.1111" hip_axis="-0.4290 0.9033 0.0000" knee_axis="0.4406 -0.8932 -0.0896" ankle_axis="0.4406 -0.8932 -0.0896" coxa_box="0.707 0.404 0.165" femur_box="0.755 0.398 0.336" foot_box="0.202 0.204 0.211"/>
+  <xacro:leg name="rf" hip="0.7292 -0.4250 0.0111" knee="0.6209 -0.2902 -0.0107" ankle="0.2435 -0.1004 0.0647" hip_axis="-0.4234 -0.9059 0.0000" knee_axis="-0.4145 -0.8932 0.1741" ankle_axis="-0.4145 -0.8932 0.1741" coxa_box="0.692 0.404 0.268" femur_box="0.782 0.398 0.204" foot_box="0.203 0.204 0.212"/>
+  <xacro:leg name="rm" hip="0.7729 0.0080 0.0299" knee="0.6838 0.0121 0.1247" ankle="0.2718 0.0053 0.0815" hip_axis="0.0178 -0.9998 0.0000" knee_axis="0.0149 -0.9998 0.0157" ankle_axis="0.0149 -0.9998 0.0157" coxa_box="0.728 0.116 0.227" femur_box="0.837 0.111 0.251" foot_box="0.202 0.202 0.215"/>
+  <xacro:leg name="rr" hip="0.7419 0.4061 -0.0572" knee="0.6345 0.2340 0.0648" ankle="0.2428 0.0751 0.1039" hip_axis="0.3460 -0.9382 0.0000" knee_axis="0.3561 -0.9192 -0.1678" ankle_axis="0.3561 -0.9192 -0.1678" coxa_box="0.697 0.377 0.338" femur_box="0.792 0.323 0.318" foot_box="0.201 0.204 0.206"/>
+  <xacro:leg name="lf" hip="-0.7421 -0.4061 0.0562" knee="-0.5934 -0.2340 0.2338" ankle="-0.2057 -0.0751 0.1656" hip_axis="-0.3668 0.9303 0.0000" knee_axis="-0.3882 0.9192 -0.0654" ankle_axis="-0.3882 0.9192 -0.0654" coxa_box="0.728 0.377 0.168" femur_box="0.717 0.323 0.495" foot_box="0.203 0.204 0.214"/>
+  <xacro:leg name="lm" hip="-0.7678 -0.0080 0.0806" knee="-0.6650 -0.0121 0.2024" ankle="-0.2607 -0.0053 0.1121" hip_axis="-0.0183 0.9998 0.0000" knee_axis="-0.0130 0.9998 0.0173" ankle_axis="-0.0130 0.9998 0.0173" coxa_box="0.723 0.116 0.192" femur_box="0.818 0.111 0.337" foot_box="0.204 0.202 0.209"/>
+  <xacro:leg name="lr" hip="-0.7200 0.4250 0.0891" knee="-0.6110 0.2902 0.1110" ankle="-0.2262 0.1004 0.1111" hip_axis="0.4290 0.9033 -0.0000" knee_axis="0.4406 0.8932 0.0896" ankle_axis="0.4406 0.8932 0.0896" coxa_box="0.707 0.404 0.165" femur_box="0.755 0.398 0.336" foot_box="0.202 0.204 0.211"/>
 </robot>

Commit message: Fix orientation (rpy=pi, suction down) + correct joint axes per part function
- flip back to rpy=pi so the suction/chassis face down and touch the ground
- joint axes per user's part description:
  hip (coxa)  = Z  (Yaw, left-right)
  knee (femur)= horizontal perpendicular to coxa (Pitch, up-down)
  foot (底盘) = horizontal along coxa (Roll, wheel axle)

File: src/zhizhu_description/urdf/zhizhu.urdf (robot description, URDF)
Before this commit: robot zhizhu, 19 links, 18 joints
Joints:
- joint ankle_lf: axis -0.3882 0.9192 -0.0654 -> -0.9303 0.3668 0.0000; limit lower=-0.78 upper=0.78 effort=30 velocity=5 -> lower=-3.14 upper=3.14 effort=30 velocity=5; origin xyz=-0.2057 -0.0751 0.1656 -> xyz=-0.2057 0.0751 -0.1656
- joint ankle_lm: axis -0.0130 0.9998 0.0173 -> -0.9998 0.0183 0.0000; limit lower=-0.78 upper=0.78 effort=30 velocity=5 -> lower=-3.14 upper=3.14 effort=30 velocity=5; origin xyz=-0.2607 -0.0053 0.1121 -> xyz=-0.2607 0.0053 -0.1121
- joint ankle_lr: axis 0.4406 0.8932 0.0896 -> -0.9033 -0.4290 0.0000; limit lower=-0.78 upper=0.78 effort=30 velocity=5 -> lower=-3.14 upper=3.14 effort=30 velocity=5; origin xyz=-0.2262 0.1004 0.1111 -> xyz=-0.2262 -0.1004 -0.1111
- joint ankle_rf: axis -0.4145 -0.8932 0.1741 -> 0.9059 0.4234 0.0000; limit lower=-0.78 upper=0.78 effort=30 velocity=5 -> lower=-3.14 upper=3.14 effort=30 velocity=5; origin xyz=0.2435 -0.1004 0.0647 -> xyz=0.2435 0.1004 -0.0647
- joint ankle_rm: axis 0.0149 -0.9998 0.0157 -> 0.9998 -0.0178 0.0000; limit lower=-0.78 upper=0.78 effort=30 velocity=5 -> lower=-3.14 upper=3.14 effort=30 velocity=5; origin xyz=0.2718 0.0053 0.0815 -> xyz=0.2718 -0.0053 -0.0815
- joint ankle_rr: axis 0.3561 -0.9192 -0.1678 -> 0.9382 -0.3460 0.0000; limit lower=-0.78 upper=0.78 effort=30 velocity=5 -> lower=-3.14 upper=3.14 effort=30 velocity=5; origin xyz=0.2428 0.0751 0.1039 -> xyz=0.2428 -0.0751 -0.1039
- joint hip_lf: axis -0.3668 0.9303 0.0000 -> 0.0000 0.0000 1.0000; origin xyz=-0.7421 -0.4061 0.0562 -> xyz=-0.7421 0.4061 -0.0562
- joint hip_lm: axis -0.0183 0.9998 0.0000 -> 0.0000 0.0000 1.0000; origin xyz=-0.7678 -0.0080 0.0806 -> xyz=-0.7678 0.0080 -0.0806
- joint hip_lr: axis 0.4290 0.9033 -0.0000 -> 0.0000 0.0000 1.0000; origin xyz=-0.7200 0.4250 0.0891 -> xyz=-0.7200 -0.4250 -0.0891
- joint hip_rf: axis -0.4234 -0.9059 0.0000 -> 0.0000 0.0000 1.0000; origin xyz=0.7292 -0.4250 0.0111 -> xyz=0.7292 0.4250 -0.0111
- joint hip_rm: axis 0.0178 -0.9998 0.0000 -> 0.0000 0.0000 1.0000; origin xyz=0.7729 0.0080 0.0299 -> xyz=0.7729 -0.0080 -0.0299
- joint hip_rr: axis 0.3460 -0.9382 0.0000 -> 0.0000 0.0000 1.0000; origin xyz=0.7419 0.4061 -0.0572 -> xyz=0.7419 -0.4061 0.0572
- joint knee_lf: axis -0.3882 0.9192 -0.0654 -> 0.3668 0.9303 -0.0000; origin xyz=-0.5934 -0.2340 0.2338 -> xyz=-0.5934 0.2340 -0.2338
- joint knee_lm: axis -0.0130 0.9998 0.0173 -> 0.0183 0.9998 -0.0000; origin xyz=-0.6650 -0.0121 0.2024 -> xyz=-0.6650 0.0121 -0.2024
- joint knee_lr: axis 0.4406 0.8932 0.0896 -> -0.4290 0.9033 0.0000; origin xyz=-0.6110 0.2902 0.1110 -> xyz=-0.6110 -0.2902 -0.1110
- joint knee_rf: axis -0.4145 -0.8932 0.1741 -> 0.4234 -0.9059 0.0000; origin xyz=0.6209 -0.2902 -0.0107 -> xyz=0.6209 0.2902 0.0107
- joint knee_rm: axis 0.0149 -0.9998 0.0157 -> -0.0178 -0.9998 0.0000; origin xyz=0.6838 0.0121 0.1247 -> xyz=0.6838 -0.0121 -0.1247
- joint knee_rr: axis 0.3561 -0.9192 -0.1678 -> -0.3460 -0.9382 0.0000; origin xyz=0.6345 0.2340 0.0648 -> xyz=0.6345 -0.2340 -0.0648

File: src/zhizhu_description/urdf/zhizhu.xacro (robot description, xacro)
@@ -20,5 +20,5 @@
     <joint name="hip_${name}" type="revolute"><parent link="body"/><child link="${name}_coxa"/><origin xyz="${hip}"/><axis xyz="${hip_axis}"/><limit lower="-1.57" upper="1.57" effort="50" velocity="5"/><dynamics damping="0.5" friction="0.5"/></joint>
     <joint name="knee_${name}" type="revolute"><parent link="${name}_coxa"/><child link="${name}_femur"/><origin xyz="${knee}"/><axis xyz="${knee_axis}"/><limit lower="-1.57" upper="1.57" effort="50" velocity="5"/><dynamics damping="0.5" friction="0.5"/></joint>
-    <joint name="ankle_${name}" type="revolute"><parent link="${name}_femur"/><child link="${name}_foot"/><origin xyz="${ankle}"/><axis xyz="${ankle_axis}"/><limit lower="-0.78" upper="0.78" effort="30" velocity="5"/><dynamics damping="0.5" friction="0.5"/></joint>
+    <joint name="ankle_${name}" type="revolute"><parent link="${name}_femur"/><child link="${name}_foot"/><origin xyz="${ankle}"/><axis xyz="${ankle_axis}"/><limit lower="-3.14" upper="3.14" effort="30" velocity="5"/><dynamics damping="0.5" friction="0.5"/></joint>
   </xacro:macro>
   <link name="body">
@@ -27,9 +27,9 @@
     <inertial><mass value="6.0"/><inertia ixx="0.4" ixy="0" ixz="0" iyy="0.35" iyz="0" izz="0.45"/></inertial>
   </link>
-  <xacro:leg name="rf" hip="0.7292 -0.4250 0.0111" knee="0.6209 -0.2902 -0.0107" ankle="0.2435 -0.1004 0.0647" hip_axis="-0.4234 -0.9059 0.0000" knee_axis="-0.4145 -0.8932 0.1741" ankle_axis="-0.4145 -0.8932 0.1741" coxa_box="0.692 0.404 0.268" femur_box="0.782 0.398 0.204" foot_box="0.203 0.204 0.212"/>
-  <xacro:leg name="rm" hip="0.7729 0.0080 0.0299" knee="0.6838 0.0121 0.1247" ankle="0.2718 0.0053 0.0815" hip_axis="0.0178 -0.9998 0.0000" knee_axis="0.0149 -0.9998 0.0157" ankle_axis="0.0149 -0.9998 0.0157" coxa_box="0.728 0.116 0.227" femur_box="0.837 0.111 0.251" foot_box="0.202 0.202 0.215"/>
-  <xacro:leg name="rr" hip="0.7419 0.4061 -0.0572" knee="0.6345 0.2340 0.0648" ankle="0.2428 0.0751 0.1039" hip_axis="0.3460 -0.9382 0.0000" knee_axis="0.3561 -0.9192 -0.1678" ankle_axis="0.3561 -0.9192 -0.1678" coxa_box="0.697 0.377 0.338" femur_box="0.792 0.323 0.318" foot_box="0.201 0.204 0.206"/>
-  <xacro:leg name="lf" hip="-0.7421 -0.4061 0.0562" knee="-0.5934 -0.2340 0.2338" ankle="-0.2057 -0.0751 0.1656" hip_axis="-0.3668 0.9303 0.0000" knee_axis="-0.3882 0.9192 -0.0654" ankle_axis="-0.3882 0.9192 -0.0654" coxa_box="0.728 0.377 0.168" femur_box="0.717 0.323 0.495" foot_box="0.203 0.204 0.214"/>
-  <xacro:leg name="lm" hip="-0.7678 -0.0080 0.0806" knee="-0.6650 -0.0121 0.2024" ankle="-0.2607 -0.0053 0.1121" hip_axis="-0.0183 0.9998 0.0000" knee_axis="-0.0130 0.9998 0.0173" ankle_axis="-0.0130 0.9998 0.0173" coxa_box="0.723 0.116 0.192" femur_box="0.818 0.111 0.337" foot_box="0.204 0.202 0.209"/>
-  <xacro:leg name="lr" hip="-0.7200 0.4250 0.0891" knee="-0.6110 0.2902 0.1110" ankle="-0.2262 0.1004 0.1111" hip_axis="0.4290 0.9033 -0.0000" knee_axis="0.4406 0.8932 0.0896" ankle_axis="0.4406 0.8932 0.0896" coxa_box="0.707 0.404 0.165" femur_box="0.755 0.398 0.336" foot_box="0.202 0.204 0.211"/>
+  <xacro:leg name="rf" hip="0.7292 0.4250 -0.0111" knee="0.6209 0.2902 0.0107" ankle="0.2435 0.1004 -0.0647" hip_axis="0.0000 0.0000 1.0000" knee_axis="0.4234 -0.9059 0.0000" ankle_axis="0.9059 0.4234 0.0000" coxa_box="0.692 0.404 0.268" femur_box="0.782 0.398 0.204" foot_box="0.203 0.204 0.212"/>
+  <xacro:leg name="rm" hip="0.7729 -0.0080 -0.0299" knee="0.6838 -0.0121 -0.1247" ankle="0.2718 -0.0053 -0.0815" hip_axis="0.0000 0.0000 1.0000" knee_axis="-0.0178 -0.9998 0.0000" ankle_axis="0.9998 -0.0178 0.0000" coxa_box="0.728 0.116 0.227" femur_box="0.837 0.111 0.251" foot_box="0.202 0.202 0.215"/>
+  <xacro:leg name="rr" hip="0.7419 -0.4061 0.0572" knee="0.6345 -0.2340 -0.0648" ankle="0.2428 -0.0751 -0.1039" hip_axis="0.0000 0.0000 1.0000" knee_axis="-0.3460 -0.9382 0.0000" ankle_axis="0.9382 -0.3460 0.0000" coxa_box="0.697 0.377 0.338" femur_box="0.792 0.323 0.318" foot_box="0.201 0.204 0.206"/>
+  <xacro:leg name="lf" hip="-0.7421 0.4061 -0.0562" knee="-0.5934 0.2340 -0.2338" ankle="-0.2057 0.0751 -0.1656" hip_axis="0.0000 0.0000 1.0000" knee_axis="0.3668 0.9303 -0.0000" ankle_axis="-0.9303 0.3668 0.0000" coxa_box="0.728 0.377 0.168" femur_box="0.717 0.323 0.495" foot_box="0.203 0.204 0.214"/>
+  <xacro:leg name="lm" hip="-0.7678 0.0080 -0.0806" knee="-0.6650 0.0121 -0.2024" ankle="-0.2607 0.0053 -0.1121" hip_axis="0.0000 0.0000 1.0000" knee_axis="0.0183 0.9998 -0.0000" ankle_axis="-0.9998 0.0183 0.0000" coxa_box="0.723 0.116 0.192" femur_box="0.818 0.111 0.337" foot_box="0.204 0.202 0.209"/>
+  <xacro:leg name="lr" hip="-0.7200 -0.4250 -0.0891" knee="-0.6110 -0.2902 -0.1110" ankle="-0.2262 -0.1004 -0.1111" hip_axis="0.0000 0.0000 1.0000" knee_axis="-0.4290 0.9033 0.0000" ankle_axis="-0.9033 -0.4290 0.0000" coxa_box="0.707 0.404 0.165" femur_box="0.755 0.398 0.336" foot_box="0.202 0.204 0.211"/>
 </robot>
