Commit message: Fix joint pivot: use connection points (hinges) instead of centroids
Computed the closest points between adjacent parts (gaps 0.5-4mm) as the real
joint hinge locations. Joint origins now sit at the hinges, and mesh origins
are offset by (centroid - hinge) so parts rotate about their actual joints
instead of detaching/swinging about the centroid.

File: src/zhizhu_description/urdf/zhizhu.urdf (robot description, URDF)
Before this commit: robot zhizhu, 19 links, 18 joints
Joints:
- joint ankle_lf: origin xyz=-0.2057 0.0751 -0.1656 -> xyz=-0.6506 0.2160 -0.3368
- joint ankle_lm: origin xyz=-0.2607 0.0053 -0.1121 -> xyz=-0.7223 0.0468 -0.1850
- joint ankle_lr: origin xyz=-0.2262 -0.1004 -0.1111 -> xyz=-0.6218 -0.3037 -0.2112
- joint ankle_rf: origin xyz=0.2435 0.1004 -0.0647 -> xyz=0.6843 0.3192 -0.0840
- joint ankle_rm: origin xyz=0.2718 -0.0053 -0.0815 -> xyz=0.7681 -0.0474 -0.1054
- joint ankle_rr: origin xyz=0.2428 -0.0751 -0.1039 -> xyz=0.6904 -0.2255 -0.1547
- joint hip_lf: origin xyz=-0.7421 0.4061 -0.0562 -> xyz=-0.3908 0.2529 0.4574
- joint hip_lm: origin xyz=-0.7678 0.0080 -0.0806 -> xyz=-0.3772 -0.0234 0.4559
- joint hip_lr: origin xyz=-0.7200 -0.4250 -0.0891 -> xyz=-0.3693 -0.2232 0.4541
- joint hip_rf: origin xyz=0.7292 0.4250 -0.0111 -> xyz=0.3304 0.2647 0.4563
- joint hip_rm: origin xyz=0.7729 -0.0080 -0.0299 -> xyz=0.3260 -0.0216 0.4551
- joint hip_rr: origin xyz=0.7419 -0.4061 0.0572 -> xyz=0.3477 -0.2588 0.4591
- joint knee_lf: origin xyz=-0.5934 0.2340 -0.2338 -> xyz=-0.5490 0.2521 0.0893
- joint knee_lm: origin xyz=-0.6650 0.0121 -0.2024 -> xyz=-0.6265 0.0103 0.0005
- joint knee_lr: origin xyz=-0.6110 -0.2902 -0.1110 -> xyz=-0.5889 -0.2758 0.1050
- joint knee_rf: origin xyz=0.6209 0.2902 0.0107 -> xyz=0.5452 0.2187 0.2207
- joint knee_rm: origin xyz=0.6838 -0.0121 -0.1247 -> xyz=0.6041 0.0354 0.0832
- joint knee_rr: origin xyz=0.6345 -0.2340 -0.0648 -> xyz=0.5621 -0.2553 0.2508

File: src/zhizhu_description/urdf/zhizhu.xacro (robot description, xacro)
@@ -2,18 +2,18 @@
 <robot name="zhizhu" xmlns:xacro="http://www.ros.org/wiki/xacro">
   <material name="zhizhu_gray"><color rgba="0.7 0.7 0.72 1.0"/></material>
-  <xacro:macro name="leg" params="name hip knee ankle hip_axis knee_axis ankle_axis coxa_box femur_box foot_box">
+  <xacro:macro name="leg" params="name hip knee ankle hip_axis knee_axis ankle_axis coxa_origin femur_origin foot_origin coxa_box femur_box foot_box">
     <link name="${name}_coxa">
-      <visual><geometry><mesh filename="file:///home/khalil/ROS/zhizhu/install/zhizhu_description/share/zhizhu_description/meshes/parts_urdf/${name}_coxa.stl"/></geometry><material name="zhizhu_gray"/></visual>
-      <collision><geometry><box size="${coxa_box}"/></geometry></collision>
+      <visual><origin xyz="${coxa_origin}"/><geometry><mesh filename="file:///home/khalil/ROS/zhizhu/install/zhizhu_description/share/zhizhu_description/meshes/parts_urdf/${name}_coxa.stl"/></geometry><material name="zhizhu_gray"/></visual>
+      <collision><origin xyz="${coxa_origin}"/><geometry><box size="${coxa_box}"/></geometry></collision>
       <inertial><mass value="1.5"/><inertia ixx="0.05" ixy="0" ixz="0" iyy="0.05" iyz="0" izz="0.05"/></inertial>
     </link>
     <link name="${name}_femur">
-      <visual><geometry><mesh filename="file:///home/khalil/ROS/zhizhu/install/zhizhu_description/share/zhizhu_description/meshes/parts_urdf/${name}_femur.stl"/></geometry><material name="zhizhu_gray"/></visual>
-      <collision><geometry><box size="${femur_box}"/></geometry></collision>
+      <visual><origin xyz="${femur_origin}"/><geometry><mesh filename="file:///home/khalil/ROS/zhizhu/install/zhizhu_description/share/zhizhu_description/meshes/parts_urdf/${name}_femur.stl"/></geometry><material name="zhizhu_gray"/></visual>
+      <collision><origin xyz="${femur_origin}"/><geometry><box size="${femur_box}"/></geometry></collision>
       <inertial><mass value="1.2"/><inertia ixx="0.04" ixy="0" ixz="0" iyy="0.04" iyz="0" izz="0.04"/></inertial>
     </link>
     <link name="${name}_foot">
-      <visual><geometry><mesh filename="file:///home/khalil/ROS/zhizhu/install/zhizhu_description/share/zhizhu_description/meshes/parts_urdf/${name}_foot.stl"/></geometry><material name="zhizhu_gray"/></visual>
-      <collision><geometry><box size="${foot_box}"/></geometry></collision>
+      <visual><origin xyz="${foot_origin}"/><geometry><mesh filename="file:///home/khalil/ROS/zhizhu/install/zhizhu_description/share/zhizhu_description/meshes/parts_urdf/${name}_foot.stl"/></geometry><material name="zhizhu_gray"/></visual>
+      <collision><origin xyz="${foot_origin}"/><geometry><box size="${foot_box}"/></geometry></collision>
       <inertial><mass value="0.8"/><inertia ixx="0.01" ixy="0" ixz="0" iyy="0.01" iyz="0" izz="0.01"/></inertial>
     </link>
@@ -23,13 +23,13 @@
   </xacro:macro>
   <link name="body">
-    <visual><geometry><mesh filename="file:///home/khalil/ROS/zhizhu/install/zhizhu_description/share/zhizhu_description/meshes/parts_urdf/body.stl"/></geometry><material name="zhizhu_gray"/></visual>
-    <collision><geometry><box size="0.782 0.700 0.442"/></geometry></collision>
+    <visual><origin xyz="-0.0226 -0.0000 0.6012"/><geometry><mesh filename="file:///home/khalil/ROS/zhizhu/install/zhizhu_description/share/zhizhu_description/meshes/parts_urdf/body.stl"/></geometry><material name="zhizhu_gray"/></visual>
+    <collision><origin xyz="-0.0226 -0.0000 0.6012"/><geometry><box size="0.782 0.700 0.442"/></geometry></collision>
     <inertial><mass value="6.0"/><inertia ixx="0.4" ixy="0" ixz="0" iyy="0.35" iyz="0" izz="0.45"/></inertial>
   </link>
-  <xacro:leg name="rf" hip="0.7292 0.4250 -0.0111" knee="0.6209 0.2902 0.0107" ankle="0.2435 0.1004 -0.0647" hip_axis="0.0000 0.0000 1.0000" knee_axis="0.4234 -0.9059 0.0000" ankle_axis="0.9059 0.4234 0.0000" coxa_box="0.692 0.404 0.268" femur_box="0.782 0.398 0.204" foot_box="0.203 0.204 0.212"/>
-  <xacro:leg name="rm" hip="0.7729 -0.0080 -0.0299" knee="0.6838 -0.0121 -0.1247" ankle="0.2718 -0.0053 -0.0815" hip_axis="0.0000 0.0000 1.0000" knee_axis="-0.0178 -0.9998 0.0000" ankle_axis="0.9998 -0.0178 0.0000" coxa_box="0.728 0.116 0.227" femur_box="0.837 0.111 0.251" foot_box="0.202 0.202 0.215"/>
-  <xacro:leg name="rr" hip="0.7419 -0.4061 0.0572" knee="0.6345 -0.2340 -0.0648" ankle="0.2428 -0.0751 -0.1039" hip_axis="0.0000 0.0000 1.0000" knee_axis="-0.3460 -0.9382 0.0000" ankle_axis="0.9382 -0.3460 0.0000" coxa_box="0.697 0.377 0.338" femur_box="0.792 0.323 0.318" foot_box="0.201 0.204 0.206"/>
-  <xacro:leg name="lf" hip="-0.7421 0.4061 -0.0562" knee="-0.5934 0.2340 -0.2338" ankle="-0.2057 0.0751 -0.1656" hip_axis="0.0000 0.0000 1.0000" knee_axis="0.3668 0.9303 -0.0000" ankle_axis="-0.9303 0.3668 0.0000" coxa_box="0.728 0.377 0.168" femur_box="0.717 0.323 0.495" foot_box="0.203 0.204 0.214"/>
-  <xacro:leg name="lm" hip="-0.7678 0.0080 -0.0806" knee="-0.6650 0.0121 -0.2024" ankle="-0.2607 0.0053 -0.1121" hip_axis="0.0000 0.0000 1.0000" knee_axis="0.0183 0.9998 -0.0000" ankle_axis="-0.9998 0.0183 0.0000" coxa_box="0.723 0.116 0.192" femur_box="0.818 0.111 0.337" foot_box="0.204 0.202 0.209"/>
-  <xacro:leg name="lr" hip="-0.7200 -0.4250 -0.0891" knee="-0.6110 -0.2902 -0.1110" ankle="-0.2262 -0.1004 -0.1111" hip_axis="0.0000 0.0000 1.0000" knee_axis="-0.4290 0.9033 0.0000" ankle_axis="-0.9033 -0.4290 0.0000" coxa_box="0.707 0.404 0.165" femur_box="0.755 0.398 0.336" foot_box="0.202 0.204 0.211"/>
+  <xacro:leg name="rf" hip="0.3304 0.2647 0.4563" knee="0.5452 0.2187 0.2207" ankle="0.6843 0.3192 -0.0840" hip_axis="0.0000 0.0000 1.0000" knee_axis="0.4234 -0.9059 0.0000" ankle_axis="0.9059 0.4234 0.0000" coxa_origin="0.3762 0.1602 0.1338" femur_origin="0.4519 0.2318 -0.0762" foot_origin="0.0112 0.0129 -0.0569" coxa_box="0.692 0.404 0.268" femur_box="0.782 0.398 0.204" foot_box="0.203 0.204 0.212"/>
+  <xacro:leg name="rm" hip="0.3260 -0.0216 0.4551" knee="0.6041 0.0354 0.0832" ankle="0.7681 -0.0474 -0.1054" hip_axis="0.0000 0.0000 1.0000" knee_axis="-0.0178 -0.9998 0.0000" ankle_axis="0.9998 -0.0178 0.0000" coxa_origin="0.4242 0.0135 0.1161" femur_origin="0.5039 -0.0340 -0.0918" foot_origin="0.0076 0.0081 -0.0679" coxa_box="0.728 0.116 0.227" femur_box="0.837 0.111 0.251" foot_box="0.202 0.202 0.215"/>
+  <xacro:leg name="rr" hip="0.3477 -0.2588 0.4591" knee="0.5621 -0.2553 0.2508" ankle="0.6904 -0.2255 -0.1547" hip_axis="0.0000 0.0000 1.0000" knee_axis="-0.3460 -0.9382 0.0000" ankle_axis="0.9382 -0.3460 0.0000" coxa_origin="0.3716 -0.1473 0.1992" femur_origin="0.4440 -0.1260 -0.1164" foot_origin="-0.0037 0.0244 -0.0656" coxa_box="0.697 0.377 0.338" femur_box="0.792 0.323 0.318" foot_box="0.201 0.204 0.206"/>
+  <xacro:leg name="lf" hip="-0.3908 0.2529 0.4574" knee="-0.5490 0.2521 0.0893" ankle="-0.6506 0.2160 -0.3368" hip_axis="0.0000 0.0000 1.0000" knee_axis="0.3668 0.9303 -0.0000" ankle_axis="-0.9303 0.3668 0.0000" coxa_origin="-0.3739 0.1531 0.0876" femur_origin="-0.4183 0.1350 -0.2354" foot_origin="0.0265 -0.0059 -0.0642" coxa_box="0.728 0.377 0.168" femur_box="0.717 0.323 0.495" foot_box="0.203 0.204 0.214"/>
+  <xacro:leg name="lm" hip="-0.3772 -0.0234 0.4559" knee="-0.6265 0.0103 0.0005" ankle="-0.7223 0.0468 -0.1850" hip_axis="0.0000 0.0000 1.0000" knee_axis="0.0183 0.9998 -0.0000" ankle_axis="-0.9998 0.0183 0.0000" coxa_origin="-0.4133 0.0314 0.0647" femur_origin="-0.4518 0.0333 -0.1382" foot_origin="0.0098 -0.0081 -0.0653" coxa_box="0.723 0.116 0.192" femur_box="0.818 0.111 0.337" foot_box="0.204 0.202 0.209"/>
+  <xacro:leg name="lr" hip="-0.3693 -0.2232 0.4541" knee="-0.5889 -0.2758 0.1050" ankle="-0.6218 -0.3037 -0.2112" hip_axis="0.0000 0.0000 1.0000" knee_axis="-0.4290 0.9033 0.0000" ankle_axis="-0.9033 -0.4290 0.0000" coxa_origin="-0.3733 -0.2018 0.0580" femur_origin="-0.3955 -0.2162 -0.1580" foot_origin="0.0002 -0.0129 -0.0580" coxa_box="0.707 0.404 0.165" femur_box="0.755 0.398 0.336" foot_box="0.202 0.204 0.211"/>
 </robot>
