Commit message: Add mesh collision + physics to fix interpenetration; multi-part joints in Gazebo
- collision geometry changed from box to the actual mesh (matches visual, fixes
  parts passing through each other)
- per-part mass + box inertia + friction (feet mu=1.0 for traction)
- Gazebo world now uses revolute joints (hinge pivots) with high damping so the
  robot is simulated as a real multi-part joint structure, not a single rigid body

File: src/zhizhu_description/urdf/zhizhu.urdf (robot description, URDF)
Before this commit: robot zhizhu, 19 links, 18 joints
Links:
- link body: mass 6.0 -> 8.0; geometry collision mesh filename=file:///home/khalil/ROS/zhizhu/install/zhizhu_description/s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; visual mesh filename=file:///home/khalil/ROS/zhizhu/install/zhizhu_description/s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
- link lf_coxa: geometry collision mesh filename=file:///home/khalil/ROS/zhizhu/install/zhizhu_description/s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; visual mesh filename=file:///home/khalil/ROS/zhizhu/install/zhizhu_description/s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
- link lf_femur: mass 1.2 -> 1.0; geometry collision mesh filename=file:///home/khalil/ROS/zhizhu/install/zhizhu_description/s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; visual mesh filename=file:///home/khalil/ROS/zhizhu/install/zhizhu_description/s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
- link lf_foot: geometry collision mesh filename=file:///home/khalil/ROS/zhizhu/install/zhizhu_description/s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; visual mesh filename=file:///home/khalil/ROS/zhizhu/install/zhizhu_description/s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
- link lm_coxa: geometry collision mesh filename=file:///home/khalil/ROS/zhizhu/install/zhizhu_description/s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; visual mesh filename=file:///home/khalil/ROS/zhizhu/install/zhizhu_description/s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
- link lm_femur: mass 1.2 -> 1.0; geometry collision mesh filename=file:///home/khalil/ROS/zhizhu/install/zhizhu_description/s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; visual mesh filename=file:///home/khalil/ROS/zhizhu/install/zhizhu_description/s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
- link lm_foot: geometry collision mesh filename=file:///home/khalil/ROS/zhizhu/install/zhizhu_description/s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; visual mesh filename=file:///home/khalil/ROS/zhizhu/install/zhizhu_description/s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
- link lr_coxa: geometry collision mesh filename=file:///home/khalil/ROS/zhizhu/install/zhizhu_description/s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; visual mesh filename=file:///home/khalil/ROS/zhizhu/install/zhizhu_description/s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
- link lr_femur: mass 1.2 -> 1.0; geometry collision mesh filename=file:///home/khalil/ROS/zhizhu/install/zhizhu_description/s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; visual mesh filename=file:///home/khalil/ROS/zhizhu/install/zhizhu_description/s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
- link lr_foot: geometry collision mesh filename=file:///home/khalil/ROS/zhizhu/install/zhizhu_description/s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; visual mesh filename=file:///home/khalil/ROS/zhizhu/install/zhizhu_description/s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
- link rf_coxa: geometry collision mesh filename=file:///home/khalil/ROS/zhizhu/install/zhizhu_description/s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; visual mesh filename=file:///home/khalil/ROS/zhizhu/install/zhizhu_description/s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
- link rf_femur: mass 1.2 -> 1.0; geometry collision mesh filename=file:///home/khalil/ROS/zhizhu/install/zhizhu_description/s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; visual mesh filename=file:///home/khalil/ROS/zhizhu/install/zhizhu_description/s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
- link rf_foot: geometry collision mesh filename=file:///home/khalil/ROS/zhizhu/install/zhizhu_description/s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; visual mesh filename=file:///home/khalil/ROS/zhizhu/install/zhizhu_description/s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
- link rm_coxa: geometry collision mesh filename=file:///home/khalil/ROS/zhizhu/install/zhizhu_description/s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; visual mesh filename=file:///home/khalil/ROS/zhizhu/install/zhizhu_description/s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
- link rm_femur: mass 1.2 -> 1.0; geometry collision mesh filename=file:///home/khalil/ROS/zhizhu/install/zhizhu_description/s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; visual mesh filename=file:///home/khalil/ROS/zhizhu/install/zhizhu_description/s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
- link rm_foot: geometry collision mesh filename=file:///home/khalil/ROS/zhizhu/install/zhizhu_description/s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; visual mesh filename=file:///home/khalil/ROS/zhizhu/install/zhizhu_description/s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
- link rr_coxa: geometry collision mesh filename=file:///home/khalil/ROS/zhizhu/install/zhizhu_description/s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; visual mesh filename=file:///home/khalil/ROS/zhizhu/install/zhizhu_description/s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
- link rr_femur: mass 1.2 -> 1.0; geometry collision mesh filename=file:///home/khalil/ROS/zhizhu/install/zhizhu_description/s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; visual mesh filename=file:///home/khalil/ROS/zhizhu/install/zhizhu_description/s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
- link rr_foot: geometry collision mesh filename=file:///home/khalil/ROS/zhizhu/install/zhizhu_description/s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; visual mesh filename=file:///home/khalil/ROS/zhizhu/install/zhizhu_description/s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

File: src/zhizhu_description/urdf/zhizhu.xacro (robot description, xacro)
@@ -2,19 +2,19 @@
 <robot name="zhizhu" xmlns:xacro="http://www.ros.org/wiki/xacro">
   <material name="zhizhu_gray"><color rgba="0.7 0.7 0.72 1.0"/></material>
-  <xacro:macro name="leg" params="name hip knee ankle hip_axis knee_axis ankle_axis coxa_origin femur_origin foot_origin coxa_box femur_box foot_box">
+  <xacro:macro name="leg" params="name hip knee ankle hip_axis knee_axis ankle_axis coxa_origin femur_origin foot_origin coxa_ixx coxa_iyy coxa_izz femur_ixx femur_iyy femur_izz foot_ixx foot_iyy foot_izz">
     <link name="${name}_coxa">
       <visual><origin xyz="${coxa_origin}"/><geometry><mesh filename="file:///home/khalil/ROS/zhizhu/install/zhizhu_description/share/zhizhu_description/meshes/parts_urdf/${name}_coxa.stl"/></geometry><material name="zhizhu_gray"/></visual>
-      <collision><origin xyz="${coxa_origin}"/><geometry><box size="${coxa_box}"/></geometry></collision>
-      <inertial><mass value="1.5"/><inertia ixx="0.05" ixy="0" ixz="0" iyy="0.05" iyz="0" izz="0.05"/></inertial>
+      <collision><origin xyz="${coxa_origin}"/><geometry><mesh filename="file:///home/khalil/ROS/zhizhu/install/zhizhu_description/share/zhizhu_description/meshes/parts_urdf/${name}_coxa.stl"/></geometry></collision>
+      <inertial><mass value="1.5"/><inertia ixx="${coxa_ixx}" ixy="0" ixz="0" iyy="${coxa_iyy}" iyz="0" izz="${coxa_izz}"/></inertial>
     </link>
     <link name="${name}_femur">
       <visual><origin xyz="${femur_origin}"/><geometry><mesh filename="file:///home/khalil/ROS/zhizhu/install/zhizhu_description/share/zhizhu_description/meshes/parts_urdf/${name}_femur.stl"/></geometry><material name="zhizhu_gray"/></visual>
-      <collision><origin xyz="${femur_origin}"/><geometry><box size="${femur_box}"/></geometry></collision>
-      <inertial><mass value="1.2"/><inertia ixx="0.04" ixy="0" ixz="0" iyy="0.04" iyz="0" izz="0.04"/></inertial>
+      <collision><origin xyz="${femur_origin}"/><geometry><mesh filename="file:///home/khalil/ROS/zhizhu/install/zhizhu_description/share/zhizhu_description/meshes/parts_urdf/${name}_femur.stl"/></geometry></collision>
+      <inertial><mass value="1.0"/><inertia ixx="${femur_ixx}" ixy="0" ixz="0" iyy="${femur_iyy}" iyz="0" izz="${femur_izz}"/></inertial>
     </link>
     <link name="${name}_foot">
       <visual><origin xyz="${foot_origin}"/><geometry><mesh filename="file:///home/khalil/ROS/zhizhu/install/zhizhu_description/share/zhizhu_description/meshes/parts_urdf/${name}_foot.stl"/></geometry><material name="zhizhu_gray"/></visual>
-      <collision><origin xyz="${foot_origin}"/><geometry><box size="${foot_box}"/></geometry></collision>
-      <inertial><mass value="0.8"/><inertia ixx="0.01" ixy="0" ixz="0" iyy="0.01" iyz="0" izz="0.01"/></inertial>
+      <collision><origin xyz="${foot_origin}"/><geometry><mesh filename="file:///home/khalil/ROS/zhizhu/install/zhizhu_description/share/zhizhu_description/meshes/parts_urdf/${name}_foot.stl"/></geometry></collision>
+      <inertial><mass value="0.8"/><inertia ixx="${foot_ixx}" ixy="0" ixz="0" iyy="${foot_iyy}" iyz="0" izz="${foot_izz}"/></inertial>
     </link>
     <joint name="hip_${name}" type="revolute"><parent link="body"/><child link="${name}_coxa"/><origin xyz="${hip}"/><axis xyz="${hip_axis}"/><limit lower="-1.57" upper="1.57" effort="50" velocity="5"/><dynamics damping="0.5" friction="0.5"/></joint>
@@ -24,12 +24,12 @@
   <link name="body">
     <visual><origin xyz="-0.0226 -0.0000 0.6012"/><geometry><mesh filename="file:///home/khalil/ROS/zhizhu/install/zhizhu_description/share/zhizhu_description/meshes/parts_urdf/body.stl"/></geometry><material name="zhizhu_gray"/></visual>
-    <collision><origin xyz="-0.0226 -0.0000 0.6012"/><geometry><box size="0.782 0.700 0.442"/></geometry></collision>
-    <inertial><mass value="6.0"/><inertia ixx="0.4" ixy="0" ixz="0" iyy="0.35" iyz="0" izz="0.45"/></inertial>
+    <collision><origin xyz="-0.0226 -0.0000 0.6012"/><geometry><mesh filename="file:///home/khalil/ROS/zhizhu/install/zhizhu_description/share/zhizhu_description/meshes/parts_urdf/body.stl"/></geometry></collision>
+    <inertial><mass value="8.0"/><inertia ixx="1.5" ixy="0" ixz="0" iyy="1.2" iyz="0" izz="1.8"/></inertial>
   </link>
-  <xacro:leg name="rf" hip="0.3304 0.2647 0.4563" knee="0.5452 0.2187 0.2207" ankle="0.6843 0.3192 -0.0840" hip_axis="0.0000 0.0000 1.0000" knee_axis="0.4234 -0.9059 0.0000" ankle_axis="0.9059 0.4234 0.0000" coxa_origin="0.3762 0.1602 0.1338" femur_origin="0.4519 0.2318 -0.0762" foot_origin="0.0112 0.0129 -0.0569" coxa_box="0.692 0.404 0.268" femur_box="0.782 0.398 0.204" foot_box="0.203 0.204 0.212"/>
-  <xacro:leg name="rm" hip="0.3260 -0.0216 0.4551" knee="0.6041 0.0354 0.0832" ankle="0.7681 -0.0474 -0.1054" hip_axis="0.0000 0.0000 1.0000" knee_axis="-0.0178 -0.9998 0.0000" ankle_axis="0.9998 -0.0178 0.0000" coxa_origin="0.4242 0.0135 0.1161" femur_origin="0.5039 -0.0340 -0.0918" foot_origin="0.0076 0.0081 -0.0679" coxa_box="0.728 0.116 0.227" femur_box="0.837 0.111 0.251" foot_box="0.202 0.202 0.215"/>
-  <xacro:leg name="rr" hip="0.3477 -0.2588 0.4591" knee="0.5621 -0.2553 0.2508" ankle="0.6904 -0.2255 -0.1547" hip_axis="0.0000 0.0000 1.0000" knee_axis="-0.3460 -0.9382 0.0000" ankle_axis="0.9382 -0.3460 0.0000" coxa_origin="0.3716 -0.1473 0.1992" femur_origin="0.4440 -0.1260 -0.1164" foot_origin="-0.0037 0.0244 -0.0656" coxa_box="0.697 0.377 0.338" femur_box="0.792 0.323 0.318" foot_box="0.201 0.204 0.206"/>
-  <xacro:leg name="lf" hip="-0.3908 0.2529 0.4574" knee="-0.5490 0.2521 0.0893" ankle="-0.6506 0.2160 -0.3368" hip_axis="0.0000 0.0000 1.0000" knee_axis="0.3668 0.9303 -0.0000" ankle_axis="-0.9303 0.3668 0.0000" coxa_origin="-0.3739 0.1531 0.0876" femur_origin="-0.4183 0.1350 -0.2354" foot_origin="0.0265 -0.0059 -0.0642" coxa_box="0.728 0.377 0.168" femur_box="0.717 0.323 0.495" foot_box="0.203 0.204 0.214"/>
-  <xacro:leg name="lm" hip="-0.3772 -0.0234 0.4559" knee="-0.6265 0.0103 0.0005" ankle="-0.7223 0.0468 -0.1850" hip_axis="0.0000 0.0000 1.0000" knee_axis="0.0183 0.9998 -0.0000" ankle_axis="-0.9998 0.0183 0.0000" coxa_origin="-0.4133 0.0314 0.0647" femur_origin="-0.4518 0.0333 -0.1382" foot_origin="0.0098 -0.0081 -0.0653" coxa_box="0.723 0.116 0.192" femur_box="0.818 0.111 0.337" foot_box="0.204 0.202 0.209"/>
-  <xacro:leg name="lr" hip="-0.3693 -0.2232 0.4541" knee="-0.5889 -0.2758 0.1050" ankle="-0.6218 -0.3037 -0.2112" hip_axis="0.0000 0.0000 1.0000" knee_axis="-0.4290 0.9033 0.0000" ankle_axis="-0.9033 -0.4290 0.0000" coxa_origin="-0.3733 -0.2018 0.0580" femur_origin="-0.3955 -0.2162 -0.1580" foot_origin="0.0002 -0.0129 -0.0580" coxa_box="0.707 0.404 0.165" femur_box="0.755 0.398 0.336" foot_box="0.202 0.204 0.211"/>
+  <xacro:leg name="rf" hip="0.3304 0.2647 0.4563" knee="0.5452 0.2187 0.2207" ankle="0.6843 0.3192 -0.0840" hip_axis="0.0000 0.0000 1.0000" knee_axis="0.4234 -0.9059 0.0000" ankle_axis="0.9059 0.4234 0.0000" coxa_origin="0.3762 0.1602 0.1338" femur_origin="0.4519 0.2318 -0.0762" foot_origin="0.0112 0.0129 -0.0569" coxa_ixx="0.0294" coxa_iyy="0.0689" coxa_izz="0.0803" femur_ixx="0.0167" femur_iyy="0.0544" femur_izz="0.0641" foot_ixx="0.0058" foot_iyy="0.0058" foot_izz="0.0055"/>
+  <xacro:leg name="rm" hip="0.3260 -0.0216 0.4551" knee="0.6041 0.0354 0.0832" ankle="0.7681 -0.0474 -0.1054" hip_axis="0.0000 0.0000 1.0000" knee_axis="-0.0178 -0.9998 0.0000" ankle_axis="0.9998 -0.0178 0.0000" coxa_origin="0.4242 0.0135 0.1161" femur_origin="0.5039 -0.0340 -0.0918" foot_origin="0.0076 0.0081 -0.0679" coxa_ixx="0.0081" coxa_iyy="0.0728" coxa_izz="0.0680" femur_ixx="0.0063" femur_iyy="0.0636" femur_izz="0.0594" foot_ixx="0.0058" foot_iyy="0.0058" foot_izz="0.0055"/>
+  <xacro:leg name="rr" hip="0.3477 -0.2588 0.4591" knee="0.5621 -0.2553 0.2508" ankle="0.6904 -0.2255 -0.1547" hip_axis="0.0000 0.0000 1.0000" knee_axis="-0.3460 -0.9382 0.0000" ankle_axis="0.9382 -0.3460 0.0000" coxa_origin="0.3716 -0.1473 0.1992" femur_origin="0.4440 -0.1260 -0.1164" foot_origin="-0.0037 0.0244 -0.0656" coxa_ixx="0.0320" coxa_iyy="0.0750" coxa_izz="0.0784" femur_ixx="0.0171" femur_iyy="0.0606" femur_izz="0.0609" foot_ixx="0.0056" foot_iyy="0.0055" foot_izz="0.0054"/>
+  <xacro:leg name="lf" hip="-0.3908 0.2529 0.4574" knee="-0.5490 0.2521 0.0893" ankle="-0.6506 0.2160 -0.3368" hip_axis="0.0000 0.0000 1.0000" knee_axis="0.3668 0.9303 -0.0000" ankle_axis="-0.9303 0.3668 0.0000" coxa_origin="-0.3739 0.1531 0.0876" femur_origin="-0.4183 0.1350 -0.2354" foot_origin="0.0265 -0.0059 -0.0642" coxa_ixx="0.0213" coxa_iyy="0.0697" coxa_izz="0.0839" femur_ixx="0.0291" femur_iyy="0.0632" femur_izz="0.0515" foot_ixx="0.0058" foot_iyy="0.0058" foot_izz="0.0055"/>
+  <xacro:leg name="lm" hip="-0.3772 -0.0234 0.4559" knee="-0.6265 0.0103 0.0005" ankle="-0.7223 0.0468 -0.1850" hip_axis="0.0000 0.0000 1.0000" knee_axis="0.0183 0.9998 -0.0000" ankle_axis="-0.9998 0.0183 0.0000" coxa_origin="-0.4133 0.0314 0.0647" femur_origin="-0.4518 0.0333 -0.1382" foot_origin="0.0098 -0.0081 -0.0653" coxa_ixx="0.0063" coxa_iyy="0.0701" coxa_izz="0.0671" femur_ixx="0.0105" femur_iyy="0.0652" femur_izz="0.0568" foot_ixx="0.0056" foot_iyy="0.0057" foot_izz="0.0055"/>
+  <xacro:leg name="lr" hip="-0.3693 -0.2232 0.4541" knee="-0.5889 -0.2758 0.1050" ankle="-0.6218 -0.3037 -0.2112" hip_axis="0.0000 0.0000 1.0000" knee_axis="-0.4290 0.9033 0.0000" ankle_axis="-0.9033 -0.4290 0.0000" coxa_origin="-0.3733 -0.2018 0.0580" femur_origin="-0.3955 -0.2162 -0.1580" foot_origin="0.0002 -0.0129 -0.0580" coxa_ixx="0.0238" coxa_iyy="0.0659" coxa_izz="0.0830" femur_ixx="0.0226" femur_iyy="0.0570" femur_izz="0.0607" foot_ixx="0.0057" foot_iyy="0.0057" foot_izz="0.0055"/>
 </robot>
